Commit message: Port gazebo_models to Jazzy + Gazebo Harmonic
- coco_robo2.urdf: swap Classic plugins for Harmonic equivalents
  - gazebo_ros2_control/GazeboSystem -> gz_ros2_control/GazeboSimSystem
  - libgazebo_ros2_control.so -> gz_ros2_control-system
  - libgazebo_ros_diff_drive.so -> gz-sim-diff-drive-system
- package.xml: replace gazebo_ros/gazebo_ros2_control with
  ros_gz_sim, ros_gz_bridge, gz_ros2_control
- full_world_robo.launch.py: replace gazebo_ros launch+spawn_entity
  with ros_gz_sim gz_sim.launch.py + create; add ros_gz_bridge for
  /cmd_vel, /odom, /clock; use TimerAction for controller spawning

Co-Authored-By: Claude Sonnet 4.6 <noreply@anthropic.com>

File: gazebo_models/urdf/coco_robo2.urdf (robot description, URDF)
Before this commit: robot coco, 11 links, 10 joints
Links:
- link dummy_link: geometry collision mesh filename=package://gazebo_models/meshes/base.stl scale=0.001 0.001 0.001; visual mesh filename=package://gazebo_models/meshes/base.stl scale=0.001 0.001 0.001
- link grip1: geometry collision mesh filename=package://gazebo_models/meshes/grip1.stl scale=0.001 0.001 0.001; visual mesh filename=package://gazebo_models/meshes/grip1.stl scale=0.001 0.001 0.001
- link grip2: geometry collision mesh filename=package://gazebo_models/meshes/grip2.stl scale=0.001 0.001 0.001; visual mesh filename=package://gazebo_models/meshes/grip2.stl scale=0.001 0.001 0.001
- link m_link1: geometry collision mesh filename=package://gazebo_models/meshes/m_link1.stl scale=0.001 0.001 0.001; visual mesh filename=package://gazebo_models/meshes/m_link1.stl scale=0.001 0.001 0.001
- link m_link2: geometry collision mesh filename=package://gazebo_models/meshes/m_link2.stl scale=0.001 0.001 0.001; visual mesh filename=package://gazebo_models/meshes/m_link2.stl scale=0.001 0.001 0.001
- link m_link3: geometry collision mesh filename=package://gazebo_models/meshes/m_link3.stl scale=0.001 0.001 0.001; visual mesh filename=package://gazebo_models/meshes/m_link3.stl scale=0.001 0.001 0.001
- link wheel1: geometry collision mesh filename=package://gazebo_models/meshes/wheel1.stl scale=0.001 0.001 0.001; visual mesh filename=package://gazebo_models/meshes/wheel1.stl scale=0.001 0.001 0.001
- link wheel2: geometry collision mesh filename=package://gazebo_models/meshes/wheel2.stl scale=0.001 0.001 0.001; visual mesh filename=package://gazebo_models/meshes/wheel2.stl scale=0.001 0.001 0.001
- link wheel3: geometry collision mesh filename=package://gazebo_models/meshes/wheel3.stl scale=0.001 0.001 0.001; visual mesh filename=package://gazebo_models/meshes/wheel3.stl scale=0.001 0.001 0.001
- link wheel4: geometry collision mesh filename=package://gazebo_models/meshes/wheel4.stl scale=0.001 0.001 0.001; visual mesh filename=package://gazebo_models/meshes/wheel4.stl scale=0.001 0.001 0.001
