Commit message: Rescue uncommitted local improvements from ~/coco_robot_ros2 workspace
Carried over work that existed only in the local working tree:
- coco_arm_controller.yaml: remove duplicate ros__parameters key
  (orphaned diff-drive params kept as comments for reference)
- abs.urdf: hardcoded absolute mesh paths -> package:// URIs
- teleop_arm_node: HOME_ELBOW 0.0 (was -2.0, outside joint limits)
- teleop_wheels_node: docstring, auto-stop safety timeout
- CMakeLists: install worlds/ and rviz/ directories
- coco_config package, RViz config, basic teleop unit tests
- Dockerfile/docker-compose, helper scripts, CI workflow, pre-commit

Co-Authored-By: Claude Fable 5 <noreply@anthropic.com>

File: gazebo_models/urdf/abs.urdf (robot description, URDF)
Before this commit: robot ramp, 1 links, 0 joints
Links:
- link ramp_link: geometry collision mesh filename=package://gazebo_models/meshes/rampcoco.stl scale=0.001 0.001 0.001; visual mesh filename=package://gazebo_models/meshes/rampcoco.stl scale=0.001 0.001 0.001
