Commit message: Layer 1: z-up re-root, top-mounted arm, 4-wheel drive, JTC arm — verified in Harmonic
Model (coco_robo2.xacro replaces coco_robo2.urdf/coco.urdf/abs.urdf):
- Re-root on REP-103 base_footprint/base_link (z-up). The CAD frame is
  preserved exactly under one fixed re-rooting joint; the roll-90 spawn
  hack is gone, so odom/TF are now semantically correct for SLAM/Nav2.
- Arm bracket remounted on the chassis TOP face. The CAD export attached
  it to the bottom plate: at q=0 the arm hung 6 cm below the wheels and
  the robot literally stood on its own elbow — the hidden root cause of
  the documented 'low RTF' (0.23 measured) and 'spawn oscillation'.
- All four wheels driven via ros2_control DiffDriveController; mixed CAD
  joint orientations normalised by flipping the right-side joint axes
  (+velocity = forward on both sides).
- Arm joints continuous->revolute with real limits and damping; gripper
  pair via 2-joint JointTrajectoryController; JTC holds position on
  activation (no home-publisher hack, no free-swing window).
- Primitive collisions (chassis box, wheel cylinders); realistic wheel
  mass 0.4 kg (CAD auto-density gave 3.74 kg/wheel = 94% of robot mass).
- ramp.sdf: static model (was a 3985 kg dynamic URDF body); repositioned
  clear of the driving arena (mesh extends 4.4 m behind its origin).

World: Harmonic system plugins (incl. sensors for Layer 2), PBR colours,
SLAM obstacles. Launch: ros_gz_sim create -name/-string (the old port
used -entity, which gflags rejects fatally — spawn never worked),
/clock bridge, controller spawners.

Teleop: wheels -> TwistStamped on /diff_drive_controller/cmd_vel (Jazzy
ddc is stamped-only); arm -> JointTrajectory.

Verified headless (gz-sim 8.11): RTF 0.998 (was 0.23); rest pose flat at
z=0; 0.3 m/s drive covers 1.00 m in 3 s; yaw tracking within 13 pct
(separation multiplier tuned); arm reaches [-1.2,-0.5] exactly and
holds; gripper 0.5/-0.5 exact.

Co-Authored-By: Claude Fable 5 <noreply@anthropic.com>

File: gazebo_models/urdf/coco_robo2.xacro (robot description, xacro)
@@ -3,334 +3,349 @@
   <!--
     ═══════════════════════════════════════════════════════════════════════
-    PARAMETERS  — edit here to reconfigure the robot
+    Coco robot — Jazzy + Gazebo Harmonic model (Layer 1 rebuild)
+    The CAD export used a Y-up frame; previously the robot was spawned
+    tipped over with roll=+90 deg to compensate, which broke REP-103
+    (odom/TF semantics) and everything downstream (SLAM, Nav2, MoveIt).
+    This model re-roots the robot on a proper z-up base_link. All CAD-frame
+    link contents (meshes, inertials, joint origins) are preserved exactly
+    and mounted under a single fixed re-rooting joint base_link->chassis_link
+    (xyz 0.12 -0.08 0, rpy +90deg roll), which the SDF converter lumps away.
+    Wheel layout in base_link frame (x forward, y left, z up):
+      wheel1 = front-right   wheel2 = rear-right   (joints base_Revolute-1/-2)
+      wheel3 = front-left    wheel4 = rear-left    (joints base_Revolute-3/-4)
+    Wheels 1/2 use axis 0 0 -1 (instead of flipping the link frame) so that
+    positive joint velocity drives the robot forward on BOTH sides — the
+    mixed CAD joint orientations are normalised here, not in plugin config.
     ═══════════════════════════════════════════════════════════════════════
   -->
-  <xacro:property name="wheel_radius"     value="0.0585"/>
-  <xacro:property name="wheel_separation" value="0.274"/>
-  <xacro:property name="wheel_mass"       value="3.7358"/>
-  <xacro:property name="wheel_max_torque" value="200.0"/>
-  <xacro:property name="arm_effort"       value="1.0"/>
-  <xacro:property name="arm_velocity"     value="1.0"/>
-  <xacro:property name="arm_lower"        value="-6.28"/>
-  <xacro:property name="arm_upper"        value="6.28"/>
-  <xacro:property name="mesh_scale"       value="0.001 0.001 0.001"/>
-  <xacro:property name="pkg"              value="package://gazebo_models/meshes"/>
-  <!--
-    ═══════════════════════════════════════════════════════════════════════
-    MACRO: wheel link  (visual STL + simplified cylinder collision)
-    ═══════════════════════════════════════════════════════════════════════
+  <xacro:property name="mesh_pkg"     value="package://gazebo_models/meshes"/>
+  <xacro:property name="mesh_scale"   value="0.001 0.001 0.001"/>
+  <xacro:property name="wheel_radius" value="0.0585"/>
+  <xacro:property name="wheel_width"  value="0.04"/>
+  <!-- CAD auto-density gave 3.74 kg per wheel (94% of robot mass), which
+       dominated the dynamics and caused massive wheel slip. 0.4 kg is a
+       realistic printed wheel; inertia = solid cylinder of that mass. -->
+  <xacro:property name="wheel_mass"   value="0.4"/>
+  <xacro:property name="arm_effort"   value="10.0"/>
+  <xacro:property name="arm_velocity" value="2.0"/>
+  <material name="coco_dark_grey"><color rgba="0.25 0.25 0.25 1"/></material>
+  <material name="coco_black"><color rgba="0.05 0.05 0.05 1"/></material>
+  <material name="coco_orange"><color rgba="0.9 0.45 0.1 1"/></material>
+  <material name="coco_light_grey"><color rgba="0.7 0.7 0.7 1"/></material>
+  <!-- ════════════════════════ BASE ════════════════════════ -->
+  <link name="base_footprint"/>
+  <!-- base_link sits at axle height; wheels contact ground 0.0135 m below -->
+  <joint name="base_footprint_joint" type="fixed">
+    <origin xyz="0 0 0.0135" rpy="0 0 0"/>
+    <parent link="base_footprint"/>
+    <child link="base_link"/>
+  </joint>
+  <link name="base_link"/>
+  <!-- Re-rooting joint: maps the CAD frame (Y-up) onto the z-up base_link.
+       Derivation: new = (x_cad + 0.12, -z_cad - 0.08, y_cad), i.e. the four
+       wheel joints land at (±0.09, ±0.137, 0.045). -->
+  <joint name="chassis_joint" type="fixed">
+    <origin xyz="0.12 -0.08 0" rpy="1.5707963267948966 0 0"/>
+    <parent link="base_link"/>
+    <child link="chassis_link"/>
+  </joint>
+  <link name="chassis_link">
+    <inertial>
+      <origin xyz="-0.11999999999999998 0.03034175823095615 -0.08" rpy="0 0 0"/>
+      <mass value="1.041325435922023"/>
+      <inertia ixx="0.0037170473661447996" iyy="0.008245766799475876" izz="0.005624963316002818"
+               ixy="8.673617379884035e-19" iyz="8.673617379884035e-19" ixz="-6.938893903907228e-18"/>
+    </inertial>
+    <visual name="chassis_visual">
+      <origin xyz="0 0 0" rpy="0 0 0"/>
+      <geometry>
+        <mesh filename="${mesh_pkg}/base.stl" scale="${mesh_scale}"/>
+      </geometry>
+      <material name="coco_dark_grey"/>
+    </visual>
+    <!-- Primitive collision (mesh bbox): big RTF win over STL collision -->
+    <collision name="chassis_collision">
+      <origin xyz="-0.12 0.03 -0.08" rpy="0 0 0"/>
+      <geometry>
+        <box size="0.24 0.06 0.274"/>
+      </geometry>
+    </collision>
+  </link>
+  <!-- ════════════════════════ WHEELS ════════════════════════
+       Link frames and contents are the original CAD export; only the
+       collision geometry is replaced by a cylinder along the spin axis (z).
   -->
-  <xacro:macro name="wheel_link" params="name mesh_file">
+  <xacro:macro name="wheel_link" params="name mesh">
     <link name="${name}">
       <inertial>
-        <origin xyz="1.944e-07 1.088e-07 -0.01382" rpy="0 0 0"/>
+        <origin xyz="0 0 -0.0138190943" rpy="0 0 0"/>
         <mass value="${wheel_mass}"/>
-        <inertia ixx="0.004951" ixy="1.855e-08" ixz="4.998e-09"
-                 iyy="0.004951" iyz="1.343e-10" izz="0.007690"/>
+        <!-- solid cylinder: izz = mr^2/2, ixx = iyy = m(3r^2 + w^2)/12 -->
+        <inertia ixx="3.95e-04" iyy="3.95e-04" izz="6.85e-04"
+                 ixy="0" iyz="0" ixz="0"/>
       </inertial>
       <visual name="${name}_visual">
-        <origin xyz="2.387e-06 0.008117 0.016168" rpy="1.5707963 0 0"/>
+        <origin xyz="2.387e-06 0.008117301100053282 0.01616833941417112" rpy="1.5707963267679181 0 0"/>
         <geometry>
-          <mesh filename="${pkg}/${mesh_file}" scale="${mesh_scale}"/>
+          <mesh filename="${mesh_pkg}/${mesh}" scale="${mesh_scale}"/>
         </geometry>
+        <material name="coco_black"/>
       </visual>
       <collision name="${name}_collision">
-        <origin xyz="0 0 0" rpy="1.5707963 0 0"/>
+        <origin xyz="0 0 -0.0155" rpy="0 0 0"/>
         <geometry>
-          <cylinder radius="${wheel_radius}" length="0.04"/>
+          <cylinder radius="${wheel_radius}" length="${wheel_width}"/>
         </geometry>
       </collision>
     </link>
   </xacro:macro>
-  <!--
-    ═══════════════════════════════════════════════════════════════════════
-    BASE
-    ═══════════════════════════════════════════════════════════════════════
-  -->
-  <link name="base"/>
-  <link name="dummy_link">
-    <inertial>
-      <origin xyz="-0.12 0.03034 -0.08" rpy="0 0 0"/>
-      <mass value="1.04133"/>
-      <inertia ixx="0.003717" ixy="8.674e-19" ixz="-6.939e-18"
-               iyy="0.008246" iyz="8.674e-19" izz="0.005625"/>
-    </inertial>
-    <visual name="base_visual">
-      <origin xyz="0 0 0" rpy="0 0 0"/>
-      <geometry>
-        <mesh filename="${pkg}/base.stl" scale="${mesh_scale}"/>
-      </geometry>
-    </visual>
-    <collision name="base_collision">
-      <origin xyz="-0.12 0.03 -0.08" rpy="0 0 0"/>
-      <geometry><box size="0.30 0.10 0.28"/></geometry>
-    </collision>
-  </link>
-  <joint name="dummy_joint" type="fixed">
-    <origin xyz="0 0 0" rpy="0 0 0"/>
-    <parent link="base"/>
-    <child link="dummy_link"/>
-  </joint>
-  <!--
-    ═══════════════════════════════════════════════════════════════════════
-    WHEELS
-    ═══════════════════════════════════════════════════════════════════════
-  -->
-  <xacro:wheel_link name="wheel1" mesh_file="wheel1.stl"/>
-  <xacro:wheel_link name="wheel2" mesh_file="wheel2.stl"/>
-  <xacro:wheel_link name="wheel3" mesh_file="wheel3.stl"/>
-  <xacro:wheel_link name="wheel4" mesh_file="wheel4.stl"/>
+  <xacro:wheel_link name="wheel1" mesh="wheel1.stl"/>
+  <xacro:wheel_link name="wheel2" mesh="wheel2.stl"/>
+  <xacro:wheel_link name="wheel3" mesh="wheel3.stl"/>
+  <xacro:wheel_link name="wheel4" mesh="wheel4.stl"/>
+  <!-- Right side (wheels 1,2): CAD frame upright, axis flipped to 0 0 -1 so
+       +velocity = forward. Left side (wheels 3,4): CAD frame rolled pi,
+       axis 0 0 1 already gives +velocity = forward. -->
   <joint name="base_Revolute-1" type="continuous">
     <origin xyz="-0.03 0.045 0.057" rpy="0 0 0"/>
-    <parent link="base"/><child link="wheel1"/>
-    <axis xyz="0 0 1"/>
-    <limit effort="${wheel_max_torque}" velocity="10.0"/>
-    <dynamics damping="0.1" friction="0.1"/>
+    <parent link="chassis_link"/>
+    <child link="wheel1"/>
+    <axis xyz="0 0 -1"/>
+    <dynamics damping="0.01" friction="0.05"/>
   </joint>
   <joint name="base_Revolute-2" type="continuous">
     <origin xyz="-0.21 0.045 0.057" rpy="0 0 0"/>
-    <parent link="base"/><child link="wheel2"/>
+    <parent link="chassis_link"/>
+    <child link="wheel2"/>
+    <axis xyz="0 0 -1"/>
+    <dynamics damping="0.01" friction="0.05"/>
+  </joint>
+  <joint name="base_Revolute-3" type="continuous">
+    <origin xyz="-0.03 0.045 -0.217" rpy="3.141592653589793 0 0"/>
+    <parent link="chassis_link"/>
+    <child link="wheel3"/>
     <axis xyz="0 0 1"/>
-    <limit effort="${wheel_max_torque}" velocity="10.0"/>
-    <dynamics damping="0.1" friction="0.1"/>
-  </joint>
-  <joint name="base_Revolute-3" type="continuous">
-    <origin xyz="-0.03 0.045 -0.217" rpy="3.14159265 0 0"/>
-    <parent link="base"/><child link="wheel3"/>
+    <dynamics damping="0.01" friction="0.05"/>
+  </joint>
+  <joint name="base_Revolute-4" type="continuous">
+    <origin xyz="-0.21 0.045 -0.217" rpy="3.141592653589793 0 0"/>
+    <parent link="chassis_link"/>
+    <child link="wheel4"/>
     <axis xyz="0 0 1"/>
-    <limit effort="${wheel_max_torque}" velocity="10.0"/>
-    <dynamics damping="0.1" friction="0.1"/>
-  </joint>
-  <joint name="base_Revolute-4" type="continuous">
-    <origin xyz="-0.21 0.045 -0.217" rpy="3.14159265 0 0"/>
-    <parent link="base"/><child link="wheel4"/>
-    <axis xyz="0 0 1"/>
-    <limit effort="${wheel_max_torque}" velocity="10.0"/>
-    <dynamics damping="0.1" friction="0.1"/>
-  </joint>
-  <!--
-    ═══════════════════════════════════════════════════════════════════════
-    ARM LINKS
-    ═══════════════════════════════════════════════════════════════════════
+    <dynamics damping="0.01" friction="0.05"/>
+  </joint>
+  <!-- ════════════════════════ ARM ════════════════════════
+       3-DOF arm + 2-finger gripper. Joints are revolute with real limits
+       (the old model used continuous joints whose <limit> tags were
+       silently ignored) and damping so the arm cannot free-swing during
+       the controller activation window.
   -->
   <link name="m_link1">
     <inertial>
-      <origin xyz="-0.038541 -0.001586 0.042751" rpy="0 0 0"/>
-      <mass value="0.10502"/>
-      <inertia ixx="0.000102" ixy="-3.334e-06" ixz="9.638e-05"
-               iyy="0.000218" iyz="3.011e-06" izz="0.000131"/>
+      <origin xyz="-0.03854063080383259 -0.0015856480020825358 0.04275065515243506" rpy="0 0 0"/>
+      <mass value="0.10501532872977405"/>
+      <inertia ixx="0.00010224213087689287" iyy="0.00021767174405659022" izz="0.00013090575214547108"
+               ixy="-3.3343062572426755e-06" iyz="3.011180028965072e-06" ixz="9.638287881954372e-05"/>
     </inertial>
     <visual name="m_link1_visual">
-      <origin xyz="-0.018369 0.0025 0.029476" rpy="0 0 0"/>
-      <geometry><mesh filename="${pkg}/m_link1.stl" scale="${mesh_scale}"/></geometry>
+      <origin xyz="-0.018369053406696097 0.002499999962747097 0.029475549941264376" rpy="0 0 0"/>
+      <geometry>
+        <mesh filename="${mesh_pkg}/m_link1.stl" scale="${mesh_scale}"/>
+      </geometry>
+      <material name="coco_light_grey"/>
     </visual>
     <collision name="m_link1_collision">
-      <origin xyz="-0.018369 0.0025 0.029476" rpy="0 0 0"/>
-      <geometry><mesh filename="${pkg}/m_link1.stl" scale="${mesh_scale}"/></geometry>
+      <origin xyz="-0.018369053406696097 0.002499999962747097 0.029475549941264376" rpy="0 0 0"/>
+      <geometry>
+        <mesh filename="${mesh_pkg}/m_link1.stl" scale="${mesh_scale}"/>
+      </geometry>
     </collision>
   </link>
   <link name="m_link2">
     <inertial>
-      <origin xyz="0.066047 -0.0055 -0.000938" rpy="0 0 0"/>
-      <mass value="0.07715"/>
-      <inertia ixx="9.355e-06" ixy="-7.938e-07" ixz="2.175e-06"
-               iyy="2.710e-04" iyz="2.288e-08" izz="2.634e-04"/>
+      <origin xyz="0.06604665739982733 -0.00550001164803783 -0.0009375331400820297" rpy="0 0 0"/>
+      <mass value="0.07714503259769957"/>
+      <inertia ixx="9.355290836035222e-06" iyy="0.00027097957152510477" izz="0.0002633781068698384"
+               ixy="-7.937952985967445e-07" iyz="2.2876686443025918e-08" ixz="2.1753091556992897e-06"/>
     </inertial>
     <visual name="m_link2_visual">
-      <origin xyz="0.099808 -0.01 -0.025757" rpy="0 0.007576 0"/>
-      <geometry><mesh filename="${pkg}/m_link2.stl" scale="${mesh_scale}"/></geometry>
+      <origin xyz="0.09980773579424788 -0.010000000111758691 -0.025756860748654162" rpy="0 0.007575854115264767 0"/>
+      <geometry>
+        <mesh filename="${mesh_pkg}/m_link2.stl" scale="${mesh_scale}"/>
+      </geometry>
+      <material name="coco_orange"/>
     </visual>
     <collision name="m_link2_collision">
-      <origin xyz="0.099808 -0.01 -0.025757" rpy="0 0.007576 0"/>
-      <geometry><mesh filename="${pkg}/m_link2.stl" scale="${mesh_scale}"/></geometry>
+      <origin xyz="0.09980773579424788 -0.010000000111758691 -0.025756860748654162" rpy="0 0.007575854115264767 0"/>
+      <geometry>
+        <mesh filename="${mesh_pkg}/m_link2.stl" scale="${mesh_scale}"/>
+      </geometry>
     </collision>
   </link>
   <link name="m_link3">
     <inertial>
-      <origin xyz="0.011018 0.01 -1.994e-05" rpy="0 0 0"/>
-      <mass value="0.024129"/>
-      <inertia ixx="1.885e-06" ixy="1.356e-20" ixz="9.747e-09"
-               iyy="7.548e-06" iyz="0.0" izz="7.270e-06"/>
+      <origin xyz="0.011018238497968848 0.009999999888241292 -1.9935736369163238e-05" rpy="0 0 0"/>
+      <mass value="0.024128837009105796"/>
+      <inertia ixx="1.8845190178237389e-06" iyy="7.548306330095421e-06" izz="7.269906777337368e-06"
+               ixy="1.3559074268166147e-20" iyz="5.6005324621510986e-39" ixz="9.746960985909268e-09"/>
     </inertial>
     <visual name="m_link3_visual">
-      <origin xyz="0 0 0" rpy="-3.14159265 -0.001812 3.14159265"/>
-      <geometry><mesh filename="${pkg}/m_link3.stl" scale="${mesh_scale}"/></geometry>
+      <origin xyz="-4.49683090764097e-09 -1.1175870895385742e-10 2.7528110546626294e-09" rpy="-3.141592653589793 -0.0018119992531012543 3.141592653589793"/>
+      <geometry>
+        <mesh filename="${mesh_pkg}/m_link3.stl" scale="${mesh_scale}"/>
+      </geometry>
+      <material name="coco_light_grey"/>
     </visual>
     <collision name="m_link3_collision">
-      <origin xyz="0 0 0" rpy="-3.14159265 -0.001812 3.14159265"/>
-      <geometry><mesh filename="${pkg}/m_link3.stl" scale="${mesh_scale}"/></geometry>
+      <origin xyz="-4.49683090764097e-09 -1.1175870895385742e-10 2.7528110546626294e-09" rpy="-3.141592653589793 -0.0018119992531012543 3.141592653589793"/>
+      <geometry>
+        <mesh filename="${mesh_pkg}/m_link3.stl" scale="${mesh_scale}"/>
+      </geometry>
     </collision>
   </link>
   <link name="grip1">
     <inertial>
-      <origin xyz="0.022688 0.004041 0.006491" rpy="0 0 0"/>
-      <mass value="0.001945"/>
-      <inertia ixx="4.349e-08" ixy="-1.054e-09" ixz="-1.220e-07"
-               iyy="6.251e-07" iyz="-2.211e-10" izz="5.975e-07"/>
+      <origin xyz="0.022687836333347696 0.004041120571939869 0.006491176980784364" rpy="0 0 0"/>
+      <mass value="0.0019453742039578018"/>
+      <inertia ixx="4.348735470033379e-08" iyy="6.250592176565233e-07" izz="5.974629046405576e-07"
+               ixy="-1.0538123946724974e-09" iyz="-2.2111795926127908e-10" ixz="-1.2202969558862574e-07"/>
     </inertial>
     <visual name="grip1_visual">
-      <origin xyz="-1.359e-05 0.007500 0" rpy="-3.14159265 9.833e-09 0.001812"/>
-      <geometry><mesh filename="${pkg}/grip1.stl" scale="${mesh_scale}"/></geometry>
+      <origin xyz="-1.3593625099403983e-05 0.0074999912986458295 -1.1175870895385742e-10" rpy="-3.141592653589793 9.832692144899154e-09 0.001811999253101829"/>
+      <geometry>
+        <mesh filename="${mesh_pkg}/grip1.stl" scale="${mesh_scale}"/>
+      </geometry>
+      <material name="coco_black"/>
     </visual>
     <collision name="grip1_collision">
-      <origin xyz="-1.359e-05 0.007500 0" rpy="-3.14159265 9.833e-09 0.001812"/>
-      <geometry><mesh filename="${pkg}/grip1.stl" scale="${mesh_scale}"/></geometry>
+      <origin xyz="-1.3593625099403983e-05 0.0074999912986458295 -1.1175870895385742e-10" rpy="-3.141592653589793 9.832692144899154e-09 0.001811999253101829"/>
+      <geometry>
+        <mesh filename="${mesh_pkg}/grip1.stl" scale="${mesh_scale}"/>
+      </geometry>
     </collision>
   </link>
   <link name="grip2">
     <inertial>
-      <origin xyz="0.020573 0.004037 -0.011561" rpy="0 0 0"/>
-      <mass value="0.001945"/>
-      <inertia ixx="1.280e-07" ixy="-9.007e-10" ixz="2.336e-07"
-               iyy="6.251e-07" iyz="4.232e-10" izz="5.130e-07"/>
+      <origin xyz="0.02057296729304557 0.004037288426624359 -0.01156102460324302" rpy="0 0 0"/>
+      <mass value="0.0019453742039578018"/>
+      <inertia ixx="1.2796522234849025e-07" iyy="6.250594950268097e-07" izz="5.129847596221384e-07"
+               ixy="-9.007383940598359e-10" iyz="4.2322370849995914e-10" ixz="2.335670086952937e-07"/>
     </inertial>
     <visual name="grip2_visual">
-      <origin xyz="-9.096e-07 0.0005 0" rpy="0 0.233243 0.001812"/>
-      <geometry><mesh filename="${pkg}/grip2.stl" scale="${mesh_scale}"/></geometry>
+      <origin xyz="-9.096372686928644e-07 0.0005000027903372128 -1.1175870895385742e-10" rpy="6.964882040425079e-18 0.23324311682993576 0.001811999253101171"/>
+      <geometry>
+        <mesh filename="${mesh_pkg}/grip2.stl" scale="${mesh_scale}"/>
+      </geometry>
+      <material name="coco_black"/>
     </visual>
     <collision name="grip2_collision">
-      <origin xyz="-9.096e-07 0.0005 0" rpy="0 0.233243 0.001812"/>
-      <geometry><mesh filename="${pkg}/grip2.stl" scale="${mesh_scale}"/></geometry>
-    </collision>
-  </link>
-  <!--
-    ═══════════════════════════════════════════════════════════════════════
-    ARM JOINTS  (revolute with damping — prevents twitching)
-    ═══════════════════════════════════════════════════════════════════════
+      <origin xyz="-9.096372686928644e-07 0.0005000027903372128 -1.1175870895385742e-10" rpy="6.964882040425079e-18 0.23324311682993576 0.001811999253101171"/>
+      <geometry>
+        <mesh filename="${mesh_pkg}/grip2.stl" scale="${mesh_scale}"/>
+      </geometry>
+    </collision>
+  </link>
+  <!-- Arm mount. The CAD export attached the bracket to the chassis BOTTOM
+       face (y=0 in CAD coords, +90deg roll), which put the whole arm BELOW
+       the wheels — the robot literally stood on its elbow (this was the
+       hidden cause of the original "low RTF" and "arm oscillation" issues).
+       Remounted on the TOP face (y=0.06) with mirrored roll: shoulder pivot
+       lands at z=0.135, q=0 is a safe horizontal home, negative shoulder
+       raises the arm, small positive shoulder reaches down to the floor in
+       front of the robot (pick-and-place workspace). -->
+  <joint name="base_Rigid-5" type="fixed">
+    <origin xyz="-0.12 0.06 -0.08" rpy="-1.5707963267948966 0 0"/>
+    <parent link="chassis_link"/>
+    <child link="m_link1"/>
+  </joint>
+  <joint name="m_link1_Revolute-6" type="revolute">
+    <origin xyz="-0.075 0.0075 0.075" rpy="3.141592653589793 0 0"/>
+    <parent link="m_link1"/>
+    <child link="m_link2"/>
+    <axis xyz="0 -1 0"/>
+    <limit effort="${arm_effort}" velocity="${arm_velocity}" lower="-3.84" upper="1.0"/>
+    <dynamics damping="0.2" friction="0.1"/>
+  </joint>
+  <joint name="m_link2_Revolute-7" type="revolute">
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