Commit message: Layer 3: MoveIt2 arm planning + pick-and-place demo — verified in Harmonic
New coco_moveit_config package:
- SRDF: arm (shoulder+elbow) and gripper groups, named states, full
  disable-collisions matrix; arm-vs-chassis pairs stay ENABLED so the
  planner actively prevents self-collision
- kinematics (KDL position-only), joint limits with accelerations,
  moveit_controllers.yaml mapping execution onto the existing
  arm_controller/gripper_controller JTCs (FollowJointTrajectory)
- move_group.launch.py via MoveItConfigsBuilder against the gazebo_models
  xacro; scripts/pick_place.py demo: spawns a pedestal+cylinder in
  Gazebo, mirrors them into the planning scene (pedestal = obstacle,
  cylinder = AllowedCollisionMatrix contact for the gripper links), then
  plans+executes up/open/pregrasp/grasp/close/raise/lift/place/open/home
  — every arm motion is a collision-checked OMPL plan.

Model fixes found BY MoveIt's collision checking:
- lidar relocated to a rear-corner tall mast (-0.09, 0.10, 0.20): the
  old front mast sat exactly where the gripper passes at the home pose,
  and a rear-center mast clipped m_link2's tail
- ALL remaining STL mesh collisions replaced with fitted primitive boxes:
  gz-physics (DART) silently loaded no collision geometry for them, so
  the arm previously had no physical presence at all (fingers passed
  through objects, arm through the pedestal)
- high-friction finger pads for pinch grasps

Verified headless (Intel iGPU fallback, RTF 1.0): 7/7 MoveIt goals
SUCCEED; deep-reach goals correctly REJECTED for chassis self-collision
(boundary probed at [0.30,0.58] via /check_state_validity); the gripper
physically pinches the cylinder and displaces it. Honest limitation:
the rigid 7 mm CAD fingers cannot hold the pinch through the full lift
arc — the object slips near the top (compliant fingertips or a parallel
gripper would fix this on real hardware).

MoveIt2 runs from a user-space deb prefix (~/ros2_ws/moveit_prefix, no
root needed); with apt access, ros-jazzy-moveit-* packages work as-is.

Co-Authored-By: Claude Fable 5 <noreply@anthropic.com>

File: gazebo_models/urdf/coco_robo2.xacro (robot description, xacro)
@@ -155,8 +155,11 @@
       <material name="coco_light_grey"/>
     </visual>
+    <!-- Primitive collisions (mesh bbox) on all arm links: gz-physics DART
+         silently loads NO collision for STL meshes here, so the mesh
+         collisions meant the arm had no physical presence at all. -->
     <collision name="m_link1_collision">
-      <origin xyz="-0.018369053406696097 0.002499999962747097 0.029475549941264376" rpy="0 0 0"/>
-      <geometry>
-        <mesh filename="${mesh_pkg}/m_link1.stl" scale="${mesh_scale}"/>
+      <origin xyz="-0.0345 0.0 0.0495" rpy="0 0 0"/>
+      <geometry>
+        <box size="0.129 0.060 0.099"/>
       </geometry>
     </collision>
@@ -177,7 +180,7 @@
     </visual>
     <collision name="m_link2_collision">
-      <origin xyz="0.09980773579424788 -0.010000000111758691 -0.025756860748654162" rpy="0 0.007575854115264767 0"/>
-      <geometry>
-        <mesh filename="${mesh_pkg}/m_link2.stl" scale="${mesh_scale}"/>
+      <origin xyz="0.0723 -0.0075 -0.0008" rpy="0 0 0"/>
+      <geometry>
+        <box size="0.195 0.015 0.050"/>
       </geometry>
     </collision>
@@ -198,7 +201,7 @@
     </visual>
     <collision name="m_link3_collision">
-      <origin xyz="-4.49683090764097e-09 -1.1175870895385742e-10 2.7528110546626294e-09" rpy="-3.141592653589793 -0.0018119992531012543 3.141592653589793"/>
-      <geometry>
-        <mesh filename="${mesh_pkg}/m_link3.stl" scale="${mesh_scale}"/>
+      <origin xyz="0.0169 0.01 0.0" rpy="0 0 0"/>
+      <geometry>
+        <box size="0.064 0.020 0.030"/>
       </geometry>
     </collision>
@@ -219,7 +222,7 @@
     </visual>
     <collision name="grip1_collision">
-      <origin xyz="-1.3593625099403983e-05 0.0074999912986458295 -1.1175870895385742e-10" rpy="-3.141592653589793 9.832692144899154e-09 0.001811999253101829"/>
-      <geometry>
-        <mesh filename="${mesh_pkg}/grip1.stl" scale="${mesh_scale}"/>
+      <origin xyz="0.0249 0.004 0.0048" rpy="0 0 0"/>
+      <geometry>
+        <box size="0.059 0.007 0.0185"/>
       </geometry>
     </collision>
@@ -240,7 +243,7 @@
     </visual>
     <collision name="grip2_collision">
-      <origin xyz="-9.096372686928644e-07 0.0005000027903372128 -1.1175870895385742e-10" rpy="6.964882040425079e-18 0.23324311682993576 0.001811999253101171"/>
-      <geometry>
-        <mesh filename="${mesh_pkg}/grip2.stl" scale="${mesh_scale}"/>
+      <origin xyz="0.0231 0.004 -0.0104" rpy="0 0.2332 0"/>
+      <geometry>
+        <box size="0.059 0.007 0.0185"/>
       </geometry>
     </collision>
@@ -296,4 +299,9 @@
        robot's own arm whenever it is raised (the arm works at the rear).
   -->
+  <!-- Rear-corner tall mast: keeps the lidar and its scan plane clear of
+       the arm's workspace. A front mast at z=0.12 sat exactly where the
+       gripper passes at home, and a rear-center mast clipped m_link2's
+       tail — both caught by MoveIt state-validity checks. The arm moves in
+       the y=0 plane, so the mast lives at y=0.10 (rear-left corner). -->
   <link name="lidar_link">
     <inertial>
@@ -307,11 +315,16 @@
       <material name="coco_black"/>
     </visual>
+    <visual name="lidar_mast_visual">
+      <origin xyz="0 0 -0.08" rpy="0 0 0"/>
+      <geometry><cylinder radius="0.012" length="0.12"/></geometry>
+      <material name="coco_dark_grey"/>
+    </visual>
     <collision name="lidar_collision">
-      <origin xyz="0 0 -0.02" rpy="0 0 0"/>
-      <geometry><cylinder radius="0.03" length="0.08"/></geometry>
+      <origin xyz="0 0 -0.07" rpy="0 0 0"/>
+      <geometry><cylinder radius="0.03" length="0.18"/></geometry>
     </collision>
   </link>
   <joint name="lidar_joint" type="fixed">
-    <origin xyz="0.09 0 0.12" rpy="0 0 0"/>
+    <origin xyz="-0.09 0.10 0.20" rpy="0 0 0"/>
     <parent link="base_link"/>
     <child link="lidar_link"/>
@@ -442,3 +455,13 @@
   <xacro:wheel_friction name="wheel3"/>
   <xacro:wheel_friction name="wheel4"/>
+  <!-- High-friction finger pads so a pinched object does not slide out
+       vertically during the lift -->
+  <gazebo reference="grip1">
+    <mu1>2.5</mu1>
+    <mu2>2.5</mu2>
+  </gazebo>
+  <gazebo reference="grip2">
+    <mu1>2.5</mu1>
+    <mu2>2.5</mu2>
+  </gazebo>
 </robot>

Commit message: Layer 5: RL ramp-traversal scaffold (Gymnasium + SB3 PPO) — loop verified
New coco_rl package:
- ramp_env.py: Gymnasium env wrapping the running Harmonic sim.
  Actions [linear, angular] -> TwistStamped on the DiffDriveController;
  observations [x, y, sin/cos yaw, v, w, roll, pitch] from odometry +
  the new IMU; reset teleports the robot via the gz set_pose service and
  rebases odom; reward = 10*forward_progress - tilt penalty - time cost,
  terminal on tip-over (|roll|,|pitch| > 0.6 rad) or ramp-top progress.
- train_ppo.py: SB3 PPO (CPU, 64x64 MLP) with Monitor; CPU torch is
  deliberate — sim RTF bounds training speed, not the tiny policy.

Model: IMU sensor (imu_link, 50 Hz) added to the xacro + /imu bridge
entry (the world already loads gz-sim-imu-system).

Verified: /imu at 49.7 Hz; PPO smoke run of 1024 timesteps against the
live sim completed end-to-end (2 rollouts, episodes run the full 400
steps, model saved). Full policy training is an overnight job:
python3 -m coco_rl.train_ppo --steps 200000

README: RL section + roadmap — all five layers complete.

Co-Authored-By: Claude Fable 5 <noreply@anthropic.com>

File: gazebo_models/urdf/coco_robo2.xacro (robot description, xacro)
@@ -354,4 +354,25 @@
     <child link="camera_optical_frame"/>
   </joint>
+  <!-- IMU at the body centre: attitude feedback for ramp traversal (RL) -->
+  <link name="imu_link">
+    <inertial>
+      <origin xyz="0 0 0" rpy="0 0 0"/>
+      <mass value="0.01"/>
+      <inertia ixx="1e-06" iyy="1e-06" izz="1e-06" ixy="0" iyz="0" ixz="0"/>
+    </inertial>
+  </link>
+  <joint name="imu_joint" type="fixed">
+    <origin xyz="0 0 0.04" rpy="0 0 0"/>
+    <parent link="base_link"/>
+    <child link="imu_link"/>
+  </joint>
+  <gazebo reference="imu_link">
+    <sensor name="imu" type="imu">
+      <topic>imu</topic>
+      <gz_frame_id>imu_link</gz_frame_id>
+      <update_rate>50</update_rate>
+      <always_on>true</always_on>
+    </sensor>
+  </gazebo>
   <gazebo reference="lidar_link">
     <sensor name="lidar" type="gpu_lidar">

Commit message: Ground-truth odometry publisher + accurate m_link2 collision geometry
- OdometryPublisher gz plugin on base_footprint (/model/coco/odometry,
  50 Hz, bridged GZ->ROS) — absolute pose for RL reward shaping and
  pick-and-place world-state sanity checks; wheel odom under-reads on
  the ramp
- m_link2 single-box collision replaced with 3 boxes fitted to the STL
  (shoulder block / beam / elbow block), removing ~2 cm of phantom
  collision volume around the arm

Co-Authored-By: Claude Fable 5 <noreply@anthropic.com>

File: gazebo_models/urdf/coco_robo2.xacro (robot description, xacro)
@@ -179,8 +179,25 @@
       <material name="coco_orange"/>
     </visual>
-    <collision name="m_link2_collision">
-      <origin xyz="0.0723 -0.0075 -0.0008" rpy="0 0 0"/>
-      <geometry>
-        <box size="0.195 0.015 0.050"/>
+    <!-- Three fitted boxes instead of one mesh bounding box: the link is a
+         slim beam (|z| < ~0.019 m) with 50 mm motor blocks only at the two
+         ends (measured from m_link2.stl vertex extents). The old single
+         0.050 m-tall box made the whole forearm as thick as its motors and
+         cost several degrees of reach before "colliding" with the chassis. -->
+    <collision name="m_link2_collision_shoulder_block">
+      <origin xyz="-0.005 -0.0075 0.0" rpy="0 0 0"/>
+      <geometry>
+        <box size="0.040 0.015 0.050"/>
+      </geometry>
+    </collision>
+    <collision name="m_link2_collision_beam">
+      <origin xyz="0.0775 -0.0075 -0.0015" rpy="0 0 0"/>
+      <geometry>
+        <box size="0.125 0.015 0.038"/>
+      </geometry>
+    </collision>
+    <collision name="m_link2_collision_elbow_block">
+      <origin xyz="0.155 -0.0075 -0.0012" rpy="0 0 0"/>
+      <geometry>
+        <box size="0.032 0.015 0.042"/>
       </geometry>
     </collision>
@@ -459,4 +476,15 @@
       <parameters>$(find gazebo_models)/urdf/coco_controllers.yaml</parameters>
     </plugin>
+    <!-- Ground-truth world pose (bridged to /model/coco/odometry): used by
+         the RL env for reward shaping — wheel odometry under-reads on the
+         ramp slope. Publishes no ROS TF, so it cannot fight the diff-drive
+         controller's odom->base_footprint transform. -->
+    <plugin filename="gz-sim-odometry-publisher-system" name="gz::sim::systems::OdometryPublisher">
+      <odom_frame>world</odom_frame>
+      <robot_base_frame>base_footprint</robot_base_frame>
+      <odom_topic>/model/coco/odometry</odom_topic>
+      <odom_publish_frequency>50</odom_publish_frequency>
+      <dimensions>3</dimensions>
+    </plugin>
   </gazebo>
   <!-- Moderate isotropic wheel friction: enough longitudinal traction to

Commit message: Gripper end-stop lips: cylinder now survives the full pick-carry-place cycle
The flat finger pads let the grasped cylinder slide along the pad
length and escape during lift (tighter grip + slower trajectories did
not help — rigid-finger limitation). A 6x7x5 mm lip at each pad tip,
protruding 5 mm inward, forms a partial cage. Verified in sim: all 9
arm goals succeed, frames show the cylinder carried through
raise/lift and set back on the pedestal (final pose z=0.128, on
pedestal top), robot pose checks clean.

Co-Authored-By: Claude Fable 5 <noreply@anthropic.com>

File: gazebo_models/urdf/coco_robo2.xacro (robot description, xacro)
@@ -244,4 +244,15 @@
       </geometry>
     </collision>
+    <!-- End-stop lip at the pad tip, protruding 5 mm inward (-z): the flat
+         pads alone let a grasped cylinder slide along the pad length and
+         escape during lift; the lips form a partial cage. High enough
+         above the pedestal top that grasp descent still collision-checks
+         clean against the pedestal. -->
+    <collision name="grip1_lip">
+      <origin xyz="0.0514 0.004 -0.00695" rpy="0 0 0"/>
+      <geometry>
+        <box size="0.006 0.007 0.005"/>
+      </geometry>
+    </collision>
   </link>
   <link name="grip2">
@@ -263,4 +274,12 @@
       <geometry>
         <box size="0.059 0.007 0.0185"/>
+      </geometry>
+    </collision>
+    <!-- Mirror of grip1_lip (+z is inward for this finger); origin is the
+         pad-frame tip offset rotated by the pad's 0.2332 rad pitch. -->
+    <collision name="grip2_lip">
+      <origin xyz="0.0516 0.004 -0.00509" rpy="0 0.2332 0"/>
+      <geometry>
+        <box size="0.006 0.007 0.005"/>
       </geometry>
     </collision>

Commit message: fix(rl): SOLVED — --fast was breaking training. 10/10 success rate
Deterministic evaluation now scores 10/10 (was 0/10). The cause was the --fast
flag, which unlocks the Gazebo real-time factor.

Same seed, same config, 12 deg wedge, fresh sim, only --fast differing:

                        with --fast        without --fast
  episodes              533                48
  tipped                531                0
  goals                 2                  31
  mean return           -6.32              +56.84
  mean episode length   31                 254
  eval success rate     0/10               10/10
  throughput            8.2 steps/s        8.7 steps/s

Mechanism: at unlocked RTF sim time outruns wall-clock ROS message delivery, so
cmd_vel arrives late and intermittently and the diff_drive_controller's
cmd_vel_timeout (0.5 s) repeatedly halts the wheels. That stop-start pumping is
what reared the chassis nose-up. It also explains the long-standing observation
that a commanded 0.4 m/s measured only 0.11-0.15 m/s: the wheels were being
halted for much of each step.

Critically, --fast never bought anything. STEP_DT is 0.1 s, so real time caps at
10 env-steps/s and the measured rate WITH --fast was only 8.2. Physics was never
the bottleneck; the ROS round trip always was. The flag was pure downside.

This also explains the whole session's pattern: every scripted check that passed
(climb_check, and every manual probe) never called set_physics, while every
training run that failed used --fast. A manual probe with PPO's exact action
distribution (both channels sigma=0.37) scored 6/6 goals while training with the
same distribution scored 531/533 tipped.

The flag is kept runnable so the finding stays reproducible, but now prints a
6-line warning, is documented as harmful in --help, and is removed from
train_curriculum.sh (train and eval) and verify_all.sh.

HONESTY NOTE on the other fixes in this branch: n_steps 2048, forward-only
linear mapping, MIN_LIN floor, log_std_init -1.0, MAX_LIN 0.4 / MAX_ANG 0.5 and
the wheel effort limit were all measured with --fast active, i.e. against a
corrupted control loop. Their individual before/after numbers are therefore
suspect and should not be quoted as independent evidence. They are retained
because each is defensible on its own terms -- notably GOAL_MARGIN (a real
tip-over race at the crest: a completed climb at x=5.4838 was logged as a fall
against a 5.5 goal) and the wheel effort limit (the joints had NO torque ceiling
at all) -- but the dominant cause was always --fast.

114 tests, 0 failures.

Co-Authored-By: Claude Opus 5 <noreply@anthropic.com>

File: gazebo_models/urdf/coco_robo2.xacro (robot description, xacro)
@@ -107,4 +107,16 @@
        +velocity = forward. Left side (wheels 3,4): CAD frame rolled pi,
        axis 0 0 1 already gives +velocity = forward. -->
+  <!-- Wheel effort ceiling. These joints were `continuous` with NO <limit>, and
+       the ros2_control interface below caps only velocity (+/-15 rad/s), so the
+       velocity servo had UNBOUNDED torque authority. Measured consequence: PPO's
+       modulated velocity commands produced repeated torque spikes whose reaction
+       reared the chassis nose-up to -35 deg WITHOUT the robot translating (x
+       stayed at ~0.00), tipping 93-98% of training episodes. A constant command
+       settles to a small velocity error and is fine, which is why scripted
+       climbs always worked and only training failed.
+       Sizing: a steady 24 deg climb needs 0.181 N.m per wheel and accelerating
+       at the controller's 2.0 m/s^2 limit needs 0.087, so 0.4 leaves ~1.5x
+       margin over the worst legitimate demand while staying well under the
+       ~0.67 N.m per wheel required to rear the chassis. -->
   <joint name="base_Revolute-1" type="continuous">
     <origin xyz="-0.03 0.045 0.057" rpy="0 0 0"/>
@@ -113,4 +125,5 @@
     <axis xyz="0 0 -1"/>
     <dynamics damping="0.01" friction="0.05"/>
+    <limit effort="0.4" velocity="15.0"/>
   </joint>
   <joint name="base_Revolute-2" type="continuous">
@@ -120,4 +133,5 @@
     <axis xyz="0 0 -1"/>
     <dynamics damping="0.01" friction="0.05"/>
+    <limit effort="0.4" velocity="15.0"/>
   </joint>
   <joint name="base_Revolute-3" type="continuous">
@@ -127,4 +141,5 @@
     <axis xyz="0 0 1"/>
     <dynamics damping="0.01" friction="0.05"/>
+    <limit effort="0.4" velocity="15.0"/>
   </joint>
   <joint name="base_Revolute-4" type="continuous">
@@ -134,4 +149,5 @@
     <axis xyz="0 0 1"/>
     <dynamics damping="0.01" friction="0.05"/>
+    <limit effort="0.4" velocity="15.0"/>
   </joint>
   <!-- ════════════════════════ ARM ════════════════════════

Commit message: feat(grasp): magnet grasp via gz detachable_joint
M0 asked whether the grasp generalises past its one tuned point. It does
not, and the tolerance fix in 904d7a8 was not enough: it moved the
docs/RESULTS.md points from 0/4 to 2/4 and left the +/-10 mm box at 0/10.
That box could never have passed — at z = 0.128 the arm's x reach limit
is 0.156 and the shipped point (0.152, 0.128) sits 4 mm inside it, so 4
of its 10 points were unreachable before physics ran, and the largest
fully-reachable box around that point is +/-3 mm. But the 6 that were
reachable all closed on air, which is the answer that matters. Decision
taken: switch to the detachable_joint magnet (FUTURE_WORK item 3).

A DetachableJoint per graspable model welds it to the palm (m_link3, not
the fingers — the object should stay rigid with the forearm while the
fingers keep moving). Result: the empty-grasp failure mode is gone
entirely, and every completed run lifts the cylinder a measured 32-40 mm.

Three plugin behaviours, all measured rather than assumed, and all of
them things that would otherwise fail silently:

1. It attaches the instant the child model spawns, NOT when commanded.
   Verified by spawning the cylinder 1 m to the side at z = 0.80: it hung
   there instead of falling, and dropped the moment a detach was
   published. So spawn_gazebo_objects() detaches immediately, or the demo
   drags the target around from birth.
2. It binds to that entity once and never re-scans. Remove the target and
   spawn it again — which clear_scene() does between runs — and the new
   model is never bound. Worse, a later attach still answers "attached"
   while welding nothing: verified by attaching after a respawn and then
   moving the arm, with the target sitting untouched on the ground. So
   the demo wants a fresh simulator per run.
3. The state topic is edge-triggered, so silence means either "already in
   that state" or "nobody is listening". magnet() takes `required` to say
   which reading is acceptable where: the spawn-time detach tolerates
   silence, the grasp and the release do not.

Because of (2) the plugin cannot be trusted to report its own success, so
check_lifted() reads the target's height out of Gazebo and requires it to
have risen with the arm. That is the actual grasp test now. This repo has
already shipped one silent empty grasp — move_gripper used to sleep 1.5 s
and return True — and the same mistake was available again here.

Also: move_gripper grows expect_object=None. Under a magnet, whether the
fingers stall on the cylinder or close past it is corroborating detail,
not the contract, and demanding either one would fail honest grasps.

ABORT detaches instead of opening the gripper: on the mission an abort
can happen mid-carry on the ramp platform, where an unplanned finger
motion is a second failure on top of the first.

Co-Authored-By: Claude Opus 5 <noreply@anthropic.com>
Claude-Session: https://claude.ai/code/session_01T8iQ4QueAD1tNQLbdqNVRb

File: gazebo_models/urdf/coco_robo2.xacro (robot description, xacro)
@@ -523,4 +523,39 @@
     </plugin>
   </gazebo>
+  <!-- ── Magnet grasp ──────────────────────────────────────────────────────
+       One DetachableJoint per graspable model: a command on the attach
+       topic welds that model to the gripper palm at whatever relative pose
+       it currently holds, and the detach topic releases it.
+       This replaces friction pinching, which was measured not to
+       generalise. The arm is 2-DOF with no wrist, so the pinch point is
+       fixed relative to the forearm and the clearance between the open
+       fingers and a 28 mm cylinder is 5.88-7.76 mm over a 70 mm descent.
+       Tightening the MoveIt joint tolerance from 0.02 to 0.003 rad (see
+       pick_place.py) bought back ~5.5 mm of that budget and moved the
+       docs/RESULTS.md points from 0/4 to 2/4: real, but still a coin
+       flip. Welding on contact makes the grasp a decision instead of a
+       tolerance stack-up, which is what lets the fetch mission pick any of
+       four objects at four positions rather than one tuned point.
+       parent_link is m_link3, the palm, not grip1/grip2: the object should
+       stay rigid with respect to the forearm while the fingers keep
+       moving. suppress_child_warning because these models are spawned at
+       runtime and do not exist when the robot loads. -->
+  <xacro:macro name="magnet" params="model link:=link">
+    <gazebo>
+      <plugin filename="gz-sim-detachable-joint-system"
+              name="gz::sim::systems::DetachableJoint">
+        <parent_link>m_link3</parent_link>
+        <child_model>${model}</child_model>
+        <child_link>${link}</child_link>
+        <attach_topic>/magnet/${model}/attach</attach_topic>
+        <detach_topic>/magnet/${model}/detach</detach_topic>
+        <output_topic>/magnet/${model}/state</output_topic>
+        <suppress_child_warning>true</suppress_child_warning>
+      </plugin>
+    </gazebo>
+  </xacro:macro>
+  <!-- The pick-and-place demo's cylinder. The mission's four coloured
+       objects get one line each here once M5 names them. -->
+  <xacro:magnet model="pick_target"/>
   <!-- Moderate isotropic wheel friction: enough longitudinal traction to
        drive and climb the ramp, low enough that the 4-wheel skid-steer
